File: kicad/prj/yggdrasil.kicad_sch (KiCad schematic)
At the start: 56 parts, among them J1 OLED, J2 4PIN, SW1 SW_PUSH, SW10 SW_PUSH, SW11 SW_PUSH, SW12 SW_PUSH, SW13 SW_PUSH, SW14 SW_PUSH, SW15 SW_PUSH, SW16 SW_PUSH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

Commit message: Updated spacing Re-do edge cuts Some routing Diode placement Screwhole placement
Parts:
- SW1, SW10, SW11, SW12, SW13, SW14, SW15, SW16, SW17, SW18, SW2, SW3, SW4, SW5, SW6, SW7, SW8, SW9: footprint Lily58-footprint:MX_Choc_Hotswap -> yggdrasil:Cherry_MX_Choc_Hotswap_MX_Spacing
- U1: footprint Lily58-footprint:ProMicro_rev2 -> yggdrasil:ProMicro_USB_C
Connections:
- net row0: now also D3.2 (A); no longer D3.1 (K), D4.1 (K)
- net at SW3.2: now also D3.1 (K); no longer D3.2 (A)
- net at SW4.2: now also D4.1 (K); no longer D4.2 (A)
Other:
- moved on the sheet: D3, D4

Commit message: Change switch keycap spacing Add routing Add ground plane Add logo & text
Parts:
- removed J1: OLED, Lily58-footprint:OLED_4Pin, symbol Lily58:Lily58-cache-OLED
- removed JP1, JP2, JP3, JP4, JP5, JP6, JP7, JP8: Jumper_NO_Small, Lily58-footprint:Jumper, symbol Lily58:Device-Jumper_NO_Small
